Commit message: Fix Z-fighting at the top of the bumper (visual only)
Making the bumper flush put its plates entirely inside the body's visual
cylinder, with their tops exactly level with the body's top disk. Coplanar faces
Z-fight, so the top of the bumper flickered in Gazebo, and the dark bumper band
was otherwise hidden inside the full-size body.

- the body is drawn at the collision radius (0.1720 m) instead of the full
  0.1745 m, so the bumper plates show as a dark band across the front again
- the bumper plates are drawn 1 mm short at top and bottom, so none of their
  faces shares a plane with the body's

Checked from gz's own URDF->SDF output: before, the plates spanned z
0.0125..0.079 m, exactly the body's bottom and top planes; after, 0.0135..0.078,
with no shared planes. Collisions are identical to the previous commit, so the
bumper wiring cannot have changed, and test_bumper_wiring.py still passes.

Co-Authored-By: Claude Opus 5.5 <noreply@anthropic.com>

File: urdf/robot.urdf.xacro (robot description, xacro)
@@ -17,4 +17,10 @@
   <xacro:property name="bumper_center_radius" value="${bumper_face_radius - bumper_thickness/2}"/>
   <xacro:property name="body_collision_radius" value="${bumper_face_radius - bumper_lead}"/>
+  <!-- VISUAL only. The bumper plates are drawn 1 mm short at top and bottom so no
+       face of theirs lies in the same plane as the body's top or bottom face:
+       coplanar faces Z-fight (flicker) in the renderer. Since the bumper went
+       flush its plates sit inside the body outline, so their tops were exactly
+       level with the body's top disk and flickered. -->
+  <xacro:property name="bumper_visual_inset" value="0.001"/>
   <!-- One bumper facet: a thin box tangent to the body at angle 'ang' (deg from
        front), flush with the body radius. Named collision so the contact sensor
@@ -25,5 +31,5 @@
               rpy="0 0 ${(ang+90)*DEG2RAD}"/>
       <geometry>
-        <box size="${width} ${bumper_thickness} ${bumper_height}"/>
+        <box size="${width} ${bumper_thickness} ${bumper_height - 2*bumper_visual_inset}"/>
       </geometry>
       <material name="dark"/>
@@ -174,8 +180,12 @@
   </joint>
   <link name="base_link">
+    <!-- Drawn at the collision radius, not the full body radius: the bumper
+         plates sit flush with the outline, so a full-size body would hide them
+         entirely and only their coplanar tops would show, flickering. This way
+         the dark bumper band shows across the front, as on a real robot. -->
     <visual>
       <origin xyz="0 0 ${lower_cylinder_height/2}" rpy="0 0 0"/>
       <geometry>
-        <cylinder length="${lower_cylinder_height}" radius="${base_diameter/2}"/>
+        <cylinder length="${lower_cylinder_height}" radius="${body_collision_radius}"/>
       </geometry>
       <material name="grey"/>
