Commit message: Mount the LiDAR forward, at min-range from the front edge
Move the 2D LiDAR turret from centred to base_diameter/2 - lidar_min_range
forward of centre (~0.0745 m), so its minimum range lands at the front body
edge. That keeps the sensing floor at the bumper and brings a convex corner
into view a little sooner -- earlier look-ahead for following an obstacle's
shape. lidar_center_offset stays the single knob (set 0.0 for the centred
A/B baseline); added lidar_min_range and wired it into the sensor <min> so
the offset formula and the plugin can't drift apart. Everything downstream
reads the base_scan TF, so no re-mapping and the saved maps stay valid.

Co-Authored-By: Claude Opus 4.8 <noreply@anthropic.com>

File: urdf/params.xacro (robot description, xacro)
@@ -23,7 +23,16 @@
   <!-- offset = laser_puck_height/2 so the housing bottom sits at the body top -->
   <xacro:property name="laser_puck_offset" value="0.009"/>
-  <!-- oomwoo-one: the LiDAR turret is CENTERED on top of the round body (offset = 0),
-       unlike the Proscenic M6 Pro this was forked from (whose LiDAR sat ~96.5mm rearward). -->
-  <xacro:property name="lidar_center_offset" value="0.0"/>
+  <!-- 2D LiDAR minimum range; kept in sync with the sensor <min> in plugins.xacro. -->
+  <xacro:property name="lidar_min_range" value="0.1"/>
+  <!-- LiDAR fore/aft mount on the body top (base_link +x = forward). Seated so its
+       minimum range lands at the front body edge, i.e. base_diameter/2 minus
+       lidar_min_range forward of centre (about 0.0745 m here), so the sensing floor
+       sits at the bumper and a convex corner comes into view a little sooner (earlier
+       look-ahead when following an obstacle's shape). Set to 0.0 for the centred
+       turret: the A/B baseline, and how oomwoo-one shipped before this. (The Proscenic
+       M6 Pro it was forked from sat about 96.5 mm rearward.) Everything downstream
+       reads the base_scan TF, so this is a transparent move; no re-mapping, and the
+       saved maps stay valid. -->
+  <xacro:property name="lidar_center_offset" value="${base_diameter/2 - lidar_min_range}"/>
   <!-- N*m -->
   <xacro:property name="motor_stall_torque" value="0.5"/>

File: urdf/plugins.xacro (robot description, xacro)
@@ -143,5 +143,5 @@
         </scan>
         <range>
-          <min>0.1</min>
+          <min>${lidar_min_range}</min>
           <max>10.0</max>
           <resolution>0.02</resolution>

Commit message: Revert the forward LiDAR mount: it tipped the robot onto its nose
Moving the turret forward put the centre of mass ahead of the wheel axle, and
the only support behind the axle is the single rear caster -- there is no front
caster. Measured from the live URDF: CoM sits 1.6 mm BEHIND the axle with the
turret centred, and the 150 g puck at +0.0745 m shifts it +3.8 mm, to 2.2 mm
AHEAD. The robot then rests nose-down on its front body edge at
asin(floor_clearance/(base_diameter/2)) = 4.1 deg (gz reported 3.97 deg), which
tips the scan plane onto the floor ~1.1 m ahead.

That produced a phantom "wall" perpendicular to the heading that follows the
robot everywhere: in a captured scan, r*cos(bearing) is constant at 1.07 m
across -19..-63 deg, the exact signature of a floor return, and it occludes the
real geometry beyond it. Back to 0.0, with the arithmetic recorded in the
comment so a forward mount is not retried without adding a front caster first.

Co-Authored-By: Claude Opus 5 <noreply@anthropic.com>

File: urdf/params.xacro (robot description, xacro)
@@ -25,14 +25,15 @@
   <!-- 2D LiDAR minimum range; kept in sync with the sensor <min> in plugins.xacro. -->
   <xacro:property name="lidar_min_range" value="0.1"/>
-  <!-- LiDAR fore/aft mount on the body top (base_link +x = forward). Seated so its
-       minimum range lands at the front body edge, i.e. base_diameter/2 minus
-       lidar_min_range forward of centre (about 0.0745 m here), so the sensing floor
-       sits at the bumper and a convex corner comes into view a little sooner (earlier
-       look-ahead when following an obstacle's shape). Set to 0.0 for the centred
-       turret: the A/B baseline, and how oomwoo-one shipped before this. (The Proscenic
-       M6 Pro it was forked from sat about 96.5 mm rearward.) Everything downstream
-       reads the base_scan TF, so this is a transparent move; no re-mapping, and the
-       saved maps stay valid. -->
-  <xacro:property name="lidar_center_offset" value="${base_diameter/2 - lidar_min_range}"/>
+  <!-- LiDAR fore/aft mount on the body top (base_link +x = forward). KEEP AT 0.0.
+       The only support behind the wheel axle is the single rear caster (there is no
+       front caster), so the robot tips onto its front body edge as soon as the centre
+       of mass crosses x = 0, and that margin is tiny. With the turret centred the CoM
+       sits just 1.6 mm behind the axle; moving the 150 g puck forward by
+       base_diameter/2 - lidar_min_range (0.0745 m) shifts it +3.8 mm, to 2.2 mm AHEAD.
+       The robot then rests nose-down at asin(floor_clearance/(base_diameter/2)) = 4.1
+       deg, which tips the scan plane onto the floor about 1.1 m ahead: a phantom
+       "wall" that follows the robot everywhere and wrecks wall-following and scan
+       matching alike. Mounting the LiDAR forward requires a FRONT caster first. -->
+  <xacro:property name="lidar_center_offset" value="0.0"/>
   <!-- N*m -->
   <xacro:property name="motor_stall_torque" value="0.5"/>

Commit message: Move the caster to the front, and restore the forward LiDAR mount
The rear caster was the reason the forward LiDAR tipped the robot: support
behind the axle means the centre of mass has to stay behind it, and the margin
was 1.6 mm. With the caster at the front the requirement inverts -- the CoM must
stay AHEAD of the axle -- which is exactly what the forward turret provides, so
the two changes fix each other.

Measured from the generated URDF: CoM x = +7.2 mm (the caster's own 50 g moving
from -0.1445 to +0.1445 contributes ~+4.9 mm of that), wheel and caster contact
heights both -0.0125 so the robot sits level, the caster carries 5% of the
weight, and it takes 4.31 m/s^2 of forward acceleration to unload it against a
1 m/s^2 limit -- a 4.3x margin, versus the knife edge we had before.

The LiDAR is back at base_diameter/2 - lidar_min_range (0.0745 m) forward, so
its minimum range lands at the front body edge. Both params carry comments
noting they are now coupled through the balance.

Co-Authored-By: Claude Opus 5 <noreply@anthropic.com>

File: urdf/params.xacro (robot description, xacro)
@@ -10,5 +10,8 @@
   <xacro:property name="wheel_width" value="0.012"/>
   <xacro:property name="caster_diameter" value="0.025"/>
-  <!-- Caster center to base edge -->
+  <!-- Caster center to base edge. The caster sits at the FRONT (+x), like a
+       consumer vacuum: the support polygon then spans the wheel axle (x = 0)
+       forward to the caster, so the centre of mass must stay AHEAD of the axle.
+       See lidar_center_offset below, which is what puts it there. -->
   <xacro:property name="caster_inset" value="0.030"/>
   <xacro:property name="floor_clearance" value="0.0125"/>
@@ -25,15 +28,17 @@
   <!-- 2D LiDAR minimum range; kept in sync with the sensor <min> in plugins.xacro. -->
   <xacro:property name="lidar_min_range" value="0.1"/>
-  <!-- LiDAR fore/aft mount on the body top (base_link +x = forward). KEEP AT 0.0.
-       The only support behind the wheel axle is the single rear caster (there is no
-       front caster), so the robot tips onto its front body edge as soon as the centre
-       of mass crosses x = 0, and that margin is tiny. With the turret centred the CoM
-       sits just 1.6 mm behind the axle; moving the 150 g puck forward by
-       base_diameter/2 - lidar_min_range (0.0745 m) shifts it +3.8 mm, to 2.2 mm AHEAD.
-       The robot then rests nose-down at asin(floor_clearance/(base_diameter/2)) = 4.1
-       deg, which tips the scan plane onto the floor about 1.1 m ahead: a phantom
-       "wall" that follows the robot everywhere and wrecks wall-following and scan
-       matching alike. Mounting the LiDAR forward requires a FRONT caster first. -->
-  <xacro:property name="lidar_center_offset" value="0.0"/>
+  <!-- LiDAR fore/aft mount on the body top (base_link +x = forward). Seated so its
+       minimum range lands at the front body edge: base_diameter/2 - lidar_min_range
+       (about 0.0745 m) forward of centre. That puts the sensing floor at the bumper
+       and brings a convex corner into view a little sooner.
+       This offset also carries the robot's BALANCE, so do not change it in isolation.
+       The caster is at the front, so the support spans x = 0 (wheel axle) to the
+       caster and the centre of mass must stay AHEAD of the axle. The 150 g puck at
+       +0.0745 m is what puts it there: CoM = +2.2 mm with this offset, -1.6 mm with
+       the turret centred. Get it wrong and the robot rests tilted on a body edge,
+       which drops the scan plane onto the floor about a metre out and paints a
+       phantom "wall" that follows the robot everywhere. Re-check the CoM (mass x
+       position over all links, axle at x = 0) after touching this or the caster. -->
+  <xacro:property name="lidar_center_offset" value="${base_diameter/2 - lidar_min_range}"/>
   <!-- N*m -->
   <xacro:property name="motor_stall_torque" value="0.5"/>

File: urdf/robot.urdf.xacro (robot description, xacro)
@@ -136,5 +136,5 @@
     <parent link="base_link"/>
     <child link="caster_link"/>
-    <origin xyz="${caster_inset-base_diameter/2} 0 ${caster_diameter/2-floor_clearance}" rpy="0 0 0"/>
+    <origin xyz="${base_diameter/2-caster_inset} 0 ${caster_diameter/2-floor_clearance}" rpy="0 0 0"/>
   </joint>
   <link name="caster_link">

Commit message: Add rear IR beacon receivers and baffle for docking
Two receivers either side of dead astern, splayed 25 deg, at body mid-height
to match the dock's beacon, with a fin between them. They carry the mount
geometry; the signal is simulated by oomwoo_sim_support's ir_beacon_sim.

Co-Authored-By: Claude Opus 5.5 (1M context) <noreply@anthropic.com>

File: urdf/params.xacro (robot description, xacro)
@@ -71,4 +71,21 @@
        wall following. On the physical robot this maps to a ToF (sensor_msgs/Range);
        in sim it is a 1-beam sensor_msgs/LaserScan. All values below are tunable. -->
+  <!-- Rear IR beacon receivers, for docking. Two of them, splayed either side of
+       dead astern with a baffle between, so the dock's beacon is centred when
+       both read the same: the classic balance measurement. They sit at body
+       mid-height to match the beacon's height in the dock, and face BACKWARDS
+       because the robot reverses in to wash its mops.
+       ir_rx_splay_deg is the mount angle either side of astern. Wider splay
+       sharpens the balance point (the signals cross more steeply) but shrinks
+       the arc in which both receivers see the beacon at all, which is what the
+       spin-to-find search has to land in. -->
+  <xacro:property name="ir_rx_splay_deg" value="25.0"/>
+  <xacro:property name="ir_rx_fov_deg" value="50.0"/>      <!-- half-angle each -->
+  <xacro:property name="ir_rx_y" value="0.030"/>           <!-- lateral offset -->
+  <xacro:property name="ir_rx_z" value="${lower_cylinder_height/2}"/>
+  <xacro:property name="ir_rx_size" value="0.010"/>
+  <xacro:property name="ir_rx_mass" value="0.004"/>
+  <xacro:property name="ir_baffle_len" value="0.030"/>     <!-- fin, inward from the shell -->
+  <xacro:property name="ir_baffle_thick" value="0.003"/>
   <xacro:property name="range_sensor_min" value="0.02"/>          <!-- m: closest reading -->
   <xacro:property name="range_sensor_max" value="0.50"/>          <!-- m: beyond this reads as no wall -->

File: urdf/robot.urdf.xacro (robot description, xacro)
@@ -58,4 +58,52 @@
     </link>
   </xacro:macro>
+  <!-- One rear IR beacon receiver. Its +X axis is the receiver boresight, aimed
+       backwards and splayed outward by ir_rx_splay_deg. side_sign = +1 left
+       (+Y), -1 right (-Y). Nothing in Gazebo simulates an IR receiver, so the
+       signal comes from ir_beacon_sim; these links exist to carry the mount
+       geometry, which is what the bearing is computed against. -->
+  <xacro:macro name="ir_receiver" params="prefix side_sign">
+    <joint name="${prefix}_joint" type="fixed">
+      <parent link="base_link"/>
+      <child link="${prefix}_link"/>
+      <origin xyz="${-base_diameter/2 + ir_rx_size} ${side_sign * ir_rx_y} ${ir_rx_z}"
+              rpy="0 0 ${(180.0 - side_sign * ir_rx_splay_deg) * DEG2RAD}"/>
+    </joint>
+    <link name="${prefix}_link">
+      <visual>
+        <origin xyz="0 0 0" rpy="0 0 0"/>
+        <geometry>
+          <box size="${ir_rx_size} ${ir_rx_size} ${ir_rx_size}"/>
+        </geometry>
+        <material name="dark"/>
+      </visual>
+      <xacro:solid_box_inertia m="${ir_rx_mass}"
+        x="${ir_rx_size}" y="${ir_rx_size}" z="${ir_rx_size}"/>
+    </link>
+  </xacro:macro>
+  <!-- The baffle between the receivers: a fin on the centreline, filling the
+       gap between them out to the shell. It stops each receiver seeing the
+       beacon far across the centreline (past about 70 deg, with 10 mm of fin
+       behind the receivers), which the balance would otherwise misread. Nearer
+       astern the receivers' own lobes decide: both see the beacon within about
+       +-25 deg, the window the spin-to-find search has to land in. -->
+  <xacro:macro name="ir_baffle">
+    <joint name="ir_baffle_joint" type="fixed">
+      <parent link="base_link"/>
+      <child link="ir_baffle_link"/>
+      <origin xyz="${-base_diameter/2 + ir_baffle_len/2} 0 ${ir_rx_z}" rpy="0 0 0"/>
+    </joint>
+    <link name="ir_baffle_link">
+      <visual>
+        <origin xyz="0 0 0" rpy="0 0 0"/>
+        <geometry>
+          <box size="${ir_baffle_len} ${ir_baffle_thick} ${ir_rx_size * 2}"/>
+        </geometry>
+        <material name="dark"/>
+      </visual>
+      <xacro:solid_box_inertia m="${ir_rx_mass}"
+        x="${ir_baffle_len}" y="${ir_baffle_thick}" z="${ir_rx_size * 2}"/>
+    </link>
+  </xacro:macro>
   <!-- Front multizone ToF: a small forward-facing link at body mid-height, front
        center. Its +X is the depth-grid boresight; the 16x8 ray sensor is in
@@ -230,4 +278,7 @@
   </link>
   <!-- Left/right side distance sensors (short-range wall sensors) -->
+  <xacro:ir_receiver prefix="ir_rx_left" side_sign="1"/>
+  <xacro:ir_receiver prefix="ir_rx_right" side_sign="-1"/>
+  <xacro:ir_baffle/>
   <xacro:side_range_sensor prefix="range_left" side_sign="1"/>
   <xacro:side_range_sensor prefix="range_right" side_sign="-1"/>

Commit message: Make the bumper flush: a round robot that can turn in place anywhere
The bumper facets were centred ON the body radius, so they stood 5 mm proud
and their corners reached 0.1814 m against a 0.1745 m body. Consumer vacuums
are plain circles, and for a reason: a round outline can always turn in place,
which is how a robot backs out of the tightest dead end.

The facets now sit just inside the body radius, with each facet's outer corners
landing exactly on it. Measured from gz's own URDF->SDF conversion:

                                    before     after
  facets                            12         24
  outermost point of the robot      0.1814 m   0.1745 m  (= body radius)
  body collision cylinder           0.1745 m   0.1720 m
  bumper ahead of the body, worst
  angle across the front 180 deg    +5.0 mm    +2.0 mm

Flush has one trap: a body collision cylinder of the same radius as the bumper
would tie with it, and wherever the body touched first the contact sensor
(which watches only the facets) would never fire. So the body's COLLISION
cylinder is bumper_lead (2 mm) inside the facets' flat faces, which is how a
real robot is built -- the chassis sits behind the bumper shell. The body's
VISUAL stays full size, and nothing with mass moved, so the CoM is unchanged.

12 facets per side (was 6) keeps the faceting error at 0.5 mm instead of
1.9 mm, which is what makes "flush" actually round. The contact sensors derive
their collision names from bumper_facets_per_side; test_bumper_wiring.py passes
against the new model in the jazzy-dev image.

Co-Authored-By: Claude Opus 5.5 <noreply@anthropic.com>

File: urdf/params.xacro (robot description, xacro)
@@ -54,8 +54,21 @@
        (they meet at the front, 0 deg, so there is no dead-center gap). Each half is
        'bumper_facets_per_side' thin box facets, named so the contact sensors can
-       reference them; facets sit at the body radius and protrude a few mm so they
-       are the surface that touches obstacles. -->
-  <xacro:property name="bumper_facets_per_side" value="6"/>
-  <xacro:property name="bumper_thickness" value="0.010"/> <!-- radial; outer face ~5mm proud -->
+       reference them.
+       FLUSH, not proud: the facets sit just inside the body radius, with each
+       facet's outer corners landing exactly on it, so the robot's outline is a
+       plain circle of base_diameter, like every consumer vacuum. A round outline
+       is what lets a robot turn in place out of the tightest dead end; a bumper
+       standing 5 mm proud (the earlier model) made the robot 7 mm wider in front
+       than behind, and its facet corners reached 0.1814 m instead of 0.1745 m.
+       Flush has one trap. If the body's collision cylinder had the same radius as
+       the bumper, the two would tie, and wherever the body touched first the
+       contact sensor (which watches only the facets) would never fire. So the
+       body's COLLISION cylinder is bumper_lead smaller than the facets' flat outer
+       faces, which is how a real robot is built: the chassis sits behind the
+       bumper shell. The body's VISUAL stays full size.
+       12 facets per side keep the faceting error at 0.5 mm (6 gave 1.9 mm). -->
+  <xacro:property name="bumper_facets_per_side" value="12"/>
+  <xacro:property name="bumper_thickness" value="0.010"/> <!-- radial -->
+  <xacro:property name="bumper_lead" value="0.002"/> <!-- bumper face ahead of the body collision -->
   <!-- Bumper spans the FULL body cylinder height, centered on it (like a consumer
        vacuum), so a low ledge the body can hit (e.g. a bookcase bottom shelf)

File: urdf/robot.urdf.xacro (robot description, xacro)
@@ -6,9 +6,21 @@
   <xacro:include filename="materials.xacro" />
   <!-- ****************** **************** ****************** -->
+  <!-- Bumper geometry, derived. Each facet is a flat plate whose outer corners
+       sit exactly on the body radius (flush), so its flat outer face is at
+       bumper_face_radius, a fraction of a mm inside. The body's collision
+       cylinder sits bumper_lead further in, so the bumper always touches first.
+       See the bumper notes in params.xacro. -->
+  <xacro:property name="bumper_facet_width"
+                  value="${2 * (base_diameter/2) * sin(0.5 * (90.0/bumper_facets_per_side) * DEG2RAD) * 1.15}"/>
+  <xacro:property name="bumper_face_radius"
+                  value="${sqrt((base_diameter/2)**2 - (bumper_facet_width/2)**2)}"/>
+  <xacro:property name="bumper_center_radius" value="${bumper_face_radius - bumper_thickness/2}"/>
+  <xacro:property name="body_collision_radius" value="${bumper_face_radius - bumper_lead}"/>
   <!-- One bumper facet: a thin box tangent to the body at angle 'ang' (deg from
-       front), at the body radius. Named collision so the contact sensor can list it. -->
+       front), flush with the body radius. Named collision so the contact sensor
+       can list it. -->
   <xacro:macro name="bumper_facet" params="prefix idx ang width">
     <visual>
-      <origin xyz="${(base_diameter/2)*cos(ang*DEG2RAD)} ${(base_diameter/2)*sin(ang*DEG2RAD)} ${bumper_z}"
+      <origin xyz="${bumper_center_radius*cos(ang*DEG2RAD)} ${bumper_center_radius*sin(ang*DEG2RAD)} ${bumper_z}"
               rpy="0 0 ${(ang+90)*DEG2RAD}"/>
       <geometry>
@@ -18,5 +30,5 @@
     </visual>
     <collision name="${prefix}_${idx}">
-      <origin xyz="${(base_diameter/2)*cos(ang*DEG2RAD)} ${(base_diameter/2)*sin(ang*DEG2RAD)} ${bumper_z}"
+      <origin xyz="${bumper_center_radius*cos(ang*DEG2RAD)} ${bumper_center_radius*sin(ang*DEG2RAD)} ${bumper_z}"
               rpy="0 0 ${(ang+90)*DEG2RAD}"/>
       <geometry>
@@ -31,5 +43,5 @@
       <xacro:bumper_facet prefix="${prefix}" idx="${i}"
         ang="${a0 + (i + 0.5) * (90.0 / n)}"
-        width="${2 * (base_diameter/2) * sin(0.5 * (90.0/n) * DEG2RAD) * 1.15}"/>
+        width="${bumper_facet_width}"/>
       <xacro:bumper_arc prefix="${prefix}" a0="${a0}" n="${n}" i="${i + 1}"/>
     </xacro:if>
@@ -169,8 +181,10 @@
       <material name="grey"/>
     </visual>
+    <!-- Collision is bumper_lead inside the bumper face, so the bumper touches
+         first; the visual above stays at the full body radius. -->
     <collision>
       <origin xyz="0 0 ${lower_cylinder_height/2}" rpy="0 0 0"/>
       <geometry>
-        <cylinder length="${lower_cylinder_height}" radius="${base_diameter/2}"/>
+        <cylinder length="${lower_cylinder_height}" radius="${body_collision_radius}"/>
       </geometry>
     </collision>
