Commit message: One front floor camera instead of the forward stereo pair
The two forward-looking cameras become one RGB camera, front centre, as high
as the body allows (lens ~71 mm above the floor), tilted down to watch the
floor ahead and what stands on it up to about the robot's height. Obstacle
depth comes from the two front ToF sensors; what the camera adds is the floor
itself (stains, streaks, dirt the mop pushes into lines). Not looking up is
also a privacy feature.

The tilt is derived from the FoV, not tuned: the bottom edge of the view points
straight down, so no pixels are spent on the bumper. 120 deg horizontal on a
4:3 sensor is ~104.8 deg vertical, so the tilt is ~37.6 deg down and the top
edge ~14.8 deg above horizontal. Checked in headless Gazebo: the frame runs
from bare floor at the bumper to table and chair legs, nothing higher; fx
184.8 px as expected. Topics are now /camera/image and /camera/camera_info,
frame camera_optical_frame; still off unless enable_cameras:=true. Centre of
mass moves ~0.3 mm back, still ahead of the axle.

Co-Authored-By: Claude Opus 5.5 (1M context) <noreply@anthropic.com>

File: urdf/params.xacro (robot description, xacro)
@@ -135,19 +135,32 @@
   <xacro:property name="tof_front_size" value="0.012"/>            <!-- visual cube edge (m) -->
   <xacro:property name="tof_front_mass" value="0.005"/>            <!-- kg, negligible -->
-  <!-- ****************** FRONT STEREO CAMERAS (OV5647) ****************** -->
-  <!-- Two RGB cameras, front & center, flanking the ToF sensor left/right, for
-       obstacle recognition and future stereo depth. VGA, wide FoV. The stereo base
-       is small on purpose (we only need coarse obstacle depth). URDF + camera topics
-       only for now, no stereo processing yet. Each has a REP-103 optical frame
-       (z-forward, x-right, y-down) that the image is published in. Tunable. -->
+  <!-- ****************** FRONT FLOOR CAMERA (RGB) ****************** -->
+  <!-- ONE RGB camera, front & center, as high as the body allows, tilted down to
+       watch the floor ahead and whatever stands on it up to about the robot's own
+       height. It replaces a forward-looking stereo pair: obstacle depth comes from
+       the two front ToF sensors, and what a camera adds that they cannot is the
+       FLOOR itself (stains, streaks, dirt the mop pushed into lines), which is
+       best seen looking down. Not looking up is also a privacy feature.
+       The tilt is derived, not tuned: it points the BOTTOM edge of the view
+       straight down, so no pixels are spent on the robot's own bumper. With a
+       120 deg horizontal FoV on a 4:3 sensor the vertical FoV is ~104.8 deg,
+       giving a ~37.6 deg tilt and a top edge ~14.8 deg above horizontal. From
+       about 0.1 m out it sees everything up to the robot's height (~0.1 m),
+       0.2 m tall at 0.5 m, ~0.33 m at 1 m: chair and table legs, sofa bases,
+       never faces. Change the FoV and the tilt follows. NOTE that lens listings
+       often quote DIAGONAL FoV: a "120 deg" lens is then ~108 deg horizontal.
+       REP-103 optical frame (z forward, x right, y down) for the image. -->
   <xacro:property name="camera_width" value="640"/>                <!-- VGA -->
   <xacro:property name="camera_height" value="480"/>
   <xacro:property name="camera_hfov_deg" value="120.0"/>
+  <xacro:property name="camera_vfov_deg"
+    value="${2 * degrees(atan(tan(radians(camera_hfov_deg) / 2) * camera_height / camera_width))}"/>
+  <xacro:property name="camera_pitch_deg" value="${90.0 - camera_vfov_deg / 2}"/> <!-- down; bottom edge vertical -->
   <xacro:property name="camera_near" value="0.02"/>                <!-- m -->
   <xacro:property name="camera_far" value="10.0"/>                 <!-- m -->
   <xacro:property name="camera_update_rate" value="15"/>           <!-- Hz -->
-  <xacro:property name="camera_baseline" value="0.05"/>            <!-- m: compact stereo base -->
-  <xacro:property name="camera_x" value="${base_diameter/2}"/>     <!-- front surface -->
-  <xacro:property name="camera_z" value="${lower_cylinder_height/2}"/> <!-- mid-height, flanking the ToF -->
+  <xacro:property name="camera_x" value="${base_diameter/2}"/>     <!-- front surface (window) -->
+  <!-- lens centre 8 mm under the body top: ~71 mm above the floor -->
+  <xacro:property name="camera_z" value="${lower_cylinder_height - 0.008}"/>
   <xacro:property name="camera_size" value="0.010"/>               <!-- visual cube edge (m) -->
   <xacro:property name="camera_mass" value="0.005"/>               <!-- kg, negligible -->

File: urdf/plugins.xacro (robot description, xacro)
@@ -244,15 +244,15 @@
   </gazebo>
   </xacro:if>
-  <!-- One front RGB camera (OV5647-equivalent), VGA, wide FoV. gz publishes
-       gz.msgs.Image on <topic> and gz.msgs.CameraInfo on the sibling camera_info
-       topic (the /image suffix -> /camera_info); config/gz_bridge.yaml bridges both.
-       The image is stamped in the ROS optical frame. -->
-  <xacro:macro name="camera_plugin" params="side">
-    <gazebo reference="camera_${side}_link">
-      <sensor name="camera_${side}" type="camera">
-        <pose relative_to="camera_${side}_link">0 0 0 0 0 0</pose>
+  <!-- The front floor camera: RGB, VGA, wide FoV, tilted down (params.xacro).
+       gz publishes gz.msgs.Image on <topic> and gz.msgs.CameraInfo on the sibling
+       camera_info topic (the /image suffix -> /camera_info); config/gz_bridge.yaml
+       bridges both. The image is stamped in the ROS optical frame. -->
+  <xacro:macro name="camera_plugin">
+    <gazebo reference="camera_link">
+      <sensor name="camera" type="camera">
+        <pose relative_to="camera_link">0 0 0 0 0 0</pose>
         <update_rate>${camera_update_rate}</update_rate>
-        <topic>camera_${side}/image</topic>
-        <gz_frame_id>camera_${side}_optical_frame</gz_frame_id>
+        <topic>camera/image</topic>
+        <gz_frame_id>camera_optical_frame</gz_frame_id>
         <camera>
           <horizontal_fov>${camera_hfov_deg * DEG2RAD}</horizontal_fov>
@@ -266,5 +266,5 @@
             <far>${camera_far}</far>
           </clip>
-          <optical_frame_id>camera_${side}_optical_frame</optical_frame_id>
+          <optical_frame_id>camera_optical_frame</optical_frame_id>
         </camera>
         <always_on>1</always_on>
@@ -274,6 +274,5 @@
   </xacro:macro>
   <xacro:if value="${'$(arg enable_cameras)' == 'true'}">
-    <xacro:camera_plugin side="left"/>
-    <xacro:camera_plugin side="right"/>
+    <xacro:camera_plugin/>
   </xacro:if>
   <!-- IMU: 6-axis (gyro + accelerometer) at imu_link, near the body center. gz

File: urdf/robot.urdf.xacro (robot description, xacro)
@@ -145,15 +145,16 @@
     </link>
   </xacro:macro>
-  <!-- One front RGB camera flanking the ToF, plus a ROS optical frame (REP-103:
-       x right, y down, z forward) the image is published in. side_sign = +1 left
-       (+Y), -1 right (-Y). The gz camera sensor is in plugins.xacro. -->
-  <xacro:macro name="stereo_camera" params="side side_sign">
-    <joint name="camera_${side}_joint" type="fixed">
-      <parent link="base_link"/>
-      <child link="camera_${side}_link"/>
-      <origin xyz="${camera_x} ${side_sign * camera_baseline/2} ${camera_z}"
-              rpy="0 0 0"/>
-    </joint>
-    <link name="camera_${side}_link">
+  <!-- The front floor camera, tilted down by camera_pitch_deg (positive pitch
+       about +Y tips +X towards the floor), plus a ROS optical frame (REP-103:
+       x right, y down, z forward) the image is published in. The gz camera
+       sensor is in plugins.xacro. -->
+  <xacro:macro name="floor_camera">
+    <joint name="camera_joint" type="fixed">
+      <parent link="base_link"/>
+      <child link="camera_link"/>
+      <origin xyz="${camera_x} 0 ${camera_z}"
+              rpy="0 ${radians(camera_pitch_deg)} 0"/>
+    </joint>
+    <link name="camera_link">
       <visual>
         <origin xyz="0 0 0" rpy="0 0 0"/>
@@ -166,10 +167,10 @@
         x="${camera_size}" y="${camera_size}" z="${camera_size}"/>
     </link>
-    <joint name="camera_${side}_optical_joint" type="fixed">
-      <parent link="camera_${side}_link"/>
-      <child link="camera_${side}_optical_frame"/>
+    <joint name="camera_optical_joint" type="fixed">
+      <parent link="camera_link"/>
+      <child link="camera_optical_frame"/>
       <origin xyz="0 0 0" rpy="${-pi/2} 0 ${-pi/2}"/>
     </joint>
-    <link name="camera_${side}_optical_frame"/>
+    <link name="camera_optical_frame"/>
   </xacro:macro>
   <link name="base_footprint"/>
@@ -309,7 +310,6 @@
   <!-- Front multizone ToF depth sensor (front & center) -->
   <xacro:front_tof_sensor/>
-  <!-- Front stereo cameras, flanking the ToF left/right -->
-  <xacro:stereo_camera side="left" side_sign="1"/>
-  <xacro:stereo_camera side="right" side_sign="-1"/>
+  <!-- Front floor camera, top centre, tilted down -->
+  <xacro:floor_camera/>
   <!-- IMU (gyro + accelerometer), near the body center -->
   <joint name="imu_joint" type="fixed">
